Commit message: Keep up  the simulation environment with the workPC

File: franka_panda_description/robots/hand.xacro (robot description, xacro)
@@ -65,5 +65,5 @@
       <parent link="${ns}_hand"/>
       <child link="${ns}_leftfinger"/>
-      <origin xyz="0 0 0.0584" rpy="0 0 0"/>
+      <origin xyz="0 0.0095 0.0584" rpy="0 0 0"/> <!-- 0.0095-->
       <axis xyz="0 1 0"/>
       <limit effort="20" lower="0.0" upper="0.04" velocity="0.2"/>
@@ -73,5 +73,5 @@
       <parent link="${ns}_hand"/>
       <child link="${ns}_rightfinger"/>
-      <origin xyz="0 0 0.0584" rpy="0 0 0"/>
+      <origin xyz="0 -0.0095 0.0584" rpy="0 0 0"/> <!-- 0.0095-->
       <axis xyz="0 -1 0"/>
       <limit effort="20" lower="0.0" upper="0.04" velocity="0.2"/>
@@ -79,4 +79,89 @@
       <mimic joint="${ns}_finger_joint1" />
     </joint>
+    <xacro:property name="_distance1" value="0.0584"/>
+    <xacro:property name="_distance2" value="0.03626585"/><!-- 0.09466585*-->
+    <link name="${ns}_peg">
+      <visual>
+        <geometry>
+          <mesh filename="package://franka_panda_description/meshes/collision/peg.STL"/>
+        </geometry>
+        <origin xyz="0 0 0" rpy="0 0 0"/>
+      </visual>
+      <collision>
+        <origin xyz="0 0 0" rpy="0 0 0"/>
+        <geometry>
+           <mesh filename="package://franka_panda_description/meshes/collision/peg.STL"/>
+        </geometry>
+      </collision>
+      <inertial>
+        <origin rpy="0 0 0" xyz="0 0 0.01504"/>
+        <mass value="0.02264"/>
+        <inertia ixx="2.6576e-6" ixy="0.0" ixz="0.0" iyy="8.2317e-7" iyz="0.0" izz="3.6303e-6"/>
+      </inertial>
+    </link>
+<!--
+    <joint name="${ns}_pegjoint" type="revolute">
+      <parent link="${ns}_hand"/>
+      <child link="${ns}_peg"/>
+      <origin xyz="0 0 ${_distance1 + _distance2}" rpy="0 0 3.14"/>
+      <axis xyz="0 0 1"/>
+      <limit velocity="6.5" effort="1000" lower="0" upper="0" />
+    </joint>
+-->
+    <joint name="${ns}_pegjoint" type="fixed">
+<!--
+      <preserveFixedJoint>true</preserveFixedJoint>
+-->
+      <parent link="${ns}_hand"/>
+      <child link="${ns}_peg"/>
+      <origin xyz="0 0 ${_distance1 + _distance2 + 0.035}" rpy="0 3.14159265358979 0"/>
+<!--
+      <sensor name="${ns}_pegjoint_force_torque" type="force_torque">
+        <always_on>true</always_on>
+        <visualize>false</visualize>
+        <force_torque>
+          <frame>child</frame>
+          <measure_direction>child_to_parent</measure_direction>
+        </force_torque>
+        <updateRate>30.0</updateRate>
+        <topicName>/gazebo/robot/peg/ft</topicName>
+      </sensor>
+-->
+    </joint>
+<!--
+    <gazebo reference="${ns}_pegjoint">
+      <sensor name="${ns}_pegjoint_force_torque" type="force_torque">
+        <always_on>true</always_on>
+        <visualize>true</visualize>
+        <force_torque>
+          <frame>sensor</frame>
+          <measure_direction>child_to_parent</measure_direction>
+        </force_torque>
+      </sensor>
+    </gazebo>
+    <gazebo>
+      <plugin name="ft_sensor" filename="libgazebo_ros_ft_sensor.so">
+        <updateRate>30.0</updateRate>
+        <topicName>/gazebo/robot/peg/ft</topicName>
+        <jointName>panda_pegjoint</jointName>
+      </plugin>
+    </gazebo>
+    <gazebo reference="${ns}_peg">
+      <selfCollide>true</selfCollide>
+    </gazebo>
+    <gazebo reference="${ns}_peg">
+      <sensor name='${ns}_peg_contact' type='contact'>
+        <update_rate> 50 </update_rate>
+        <always_on>true</always_on>
+          <contact>
+              <collision>${ns}_peg_collision</collision>
+          </contact>
+          <plugin name="peg_bumper" filename="libgazebo_ros_bumper.so">
+            <bumperTopicName>${ns}_peg_collision</bumperTopicName>
+            <frameName>${ns}_peg</frameName>
+          </plugin>
+      </sensor>
+    </gazebo>
+-->
   </xacro:macro>
 </robot>

File: franka_panda_description/robots/panda.gazebo.xacro (robot description, xacro)
@@ -2,29 +2,29 @@
 <robot xmlns:xacro="http://www.ros.org/wiki/xacro">
     <xacro:macro name="panda_gazebo" params="robot_name load_gripper">
+      <gazebo reference="${robot_name}_joint1">
+        <implicitSpringDamper>1</implicitSpringDamper> <!-- use ERP and CFM if this tag == true -->
+        <provideFeedback>true</provideFeedback><!-- Allows joints to publish their wrench data (force-torque) via a Gazebo plugin-->
+      </gazebo>
+      <gazebo reference="${robot_name}_joint2">
+        <implicitSpringDamper>1</implicitSpringDamper>
+        <provideFeedback>true</provideFeedback>
+      </gazebo>
+      <gazebo reference="${robot_name}_joint3">
+        <implicitSpringDamper>1</implicitSpringDamper>
+        <provideFeedback>true</provideFeedback>
+      </gazebo>
+      <gazebo reference="${robot_name}_joint4">
+        <implicitSpringDamper>1</implicitSpringDamper>
+        <provideFeedback>true</provideFeedback>
+      </gazebo>
+      <gazebo reference="${robot_name}_joint5">
+        <implicitSpringDamper>1</implicitSpringDamper>
+        <provideFeedback>true</provideFeedback>
+      </gazebo>
+      <gazebo reference="${robot_name}_joint6">
+        <implicitSpringDamper>1</implicitSpringDamper>
+        <provideFeedback>true</provideFeedback>
+      </gazebo>
       <gazebo reference="${robot_name}_joint7">
-        <implicitSpringDamper>1</implicitSpringDamper>
-        <provideFeedback>true</provideFeedback>
-      </gazebo>
-      <gazebo reference="${robot_name}_joint1">
-        <implicitSpringDamper>1</implicitSpringDamper>
-        <provideFeedback>true</provideFeedback>
-      </gazebo>
-      <gazebo reference="${robot_name}_joint2">
-        <implicitSpringDamper>1</implicitSpringDamper>
-        <provideFeedback>true</provideFeedback>
-      </gazebo>
-      <gazebo reference="${robot_name}_joint3">
-        <implicitSpringDamper>1</implicitSpringDamper>
-        <provideFeedback>true</provideFeedback>
-      </gazebo>
-      <gazebo reference="${robot_name}_joint4">
-        <implicitSpringDamper>1</implicitSpringDamper>
-        <provideFeedback>true</provideFeedback>
-      </gazebo>
-      <gazebo reference="${robot_name}_joint5">
-        <implicitSpringDamper>1</implicitSpringDamper>
-        <provideFeedback>true</provideFeedback>
-      </gazebo>
-      <gazebo reference="${robot_name}_joint6">
         <implicitSpringDamper>1</implicitSpringDamper>
         <provideFeedback>true</provideFeedback>
@@ -40,5 +40,9 @@
           </gazebo>
       </xacro:if>
-    <!-- Adding FT sensor at wrist. This is not present in real robot and is used only for computing end-point effort directly, unlike in the real robot where it is estimated from the joint efforts. -->
+    <!-- Adding FT sensor at wrist. This is not present in real robot and
+     is used only for computing end-point effort directly, unlike in the
+     real robot where it is estimated from the joint efforts. -->
+<!--
+-->
     <gazebo reference="${robot_name}_joint7">
       <disableFixedJointLumping>true</disableFixedJointLumping>
@@ -59,6 +63,34 @@
       </plugin>
     </gazebo>
+ <!--
+    <gazebo reference="taskhole_to_world">
+      <disableFixedJointLumping>true</disableFixedJointLumping>
+      <sensor name="taskhole_to_world_force_torque" type="force_torque">
+        <always_on>true</always_on>
+        <visualize>false</visualize>
+        <force_torque>
+          <frame>sensor</frame>
+          <measure_direction>child_to_parent</measure_direction>
+        </force_torque>
+      </sensor>
+    </gazebo>
+    <gazebo>
+      <plugin name="ft_sensor" filename="libgazebo_ros_ft_sensor.so">
+        <updateRate>1000.0</updateRate>
+        <topicName>/gazebo/taskhole/peg/ft</topicName>
+        <jointName>taskhole_to_world</jointName>
+      </plugin>
+    </gazebo>
+-->
     <!-- Configure self collision properties per link -->
     <!-- The gripper fingers do not have this flag otherwise the gripper would not be allowed to close correctly -->
+    <gazebo reference="${robot_name}_peg">
+      <material>
+        <script>
+          <name>Gazebo/Grey</name>
+          <uri>file://media/materials/scripts/gazebo.material</uri>
+        </script>
+      </material>
+    </gazebo>
     <gazebo reference="${robot_name}_link1">
       <selfCollide>true</selfCollide>
@@ -104,7 +136,7 @@
               <collision>${robot_name}_link2_collision</collision>
           </contact>
-          <plugin name="link2_bumper" filename="libgazebo_ros_bumper.so">
-            <bumperTopicName>${robot_name}_link2_collision</bumperTopicName>
-            <frameName>${robot_name}_link2</frameName>
+          <plugin name="peg_bumper" filename="libgazebo_ros_bumper.so">
+            <bumperTopicName>${robot_name}_peg_collision</bumperTopicName>
+            <frameName>${robot_name}_peg</frameName>
           </plugin>
       </sensor>
@@ -175,4 +207,19 @@
       </sensor>
     </gazebo>
+<!--
+    <gazebo reference="${robot_name}_peg">
+      <sensor name='${robot_name}_peg_contact' type='contact'>
+        <update_rate> 50 </update_rate>
+        <always_on>true</always_on>
+          <contact>
+              <collision>${robot_name}_peg_collision</collision>
+          </contact>
+          <plugin name="peg_bumper" filename="libgazebo_ros_bumper.so">
+            <bumperTopicName>${robot_name}_peg_collision</bumperTopicName>
+            <frameName>${robot_name}_peg</frameName>
+          </plugin>
+      </sensor>
+    </gazebo>
+-->
     <gazebo reference="${robot_name}_leftfinger">
       <sensor name='${robot_name}_leftfinger_contact' type='contact'>

File: franka_panda_description/robots/panda_arm.xacro (robot description, xacro)
@@ -1,5 +1,5 @@
 <?xml version='1.0'?>
 <robot xmlns:xacro="http://www.ros.org/wiki/xacro" name="panda">
-  <xacro:macro name="panda_arm" params="arm_id:='panda' description_pkg:='franka_panda_description' connected_to:='' in_gazebo='false' xyz:='0 0 0' rpy:='0 0 0'">
+  <xacro:macro name="panda_arm" params="arm_id:='panda' description_pkg:='franka_panda_description' connected_to:='' in_gazebo='false' xyz:='-0.0 0 0' rpy:='0 0 0'">
     <!-- If using custom frame with ${connected_to} param, make sure 'world' frame exists in its TF tree -->
     <xacro:if value="${connected_to == ''}">
@@ -232,4 +232,114 @@
       <axis xyz="0 0 0"/>
     </joint>
+<!--
+    <joint name="_worktable_to_world" type="fixed">
+      <parent link="world"/>
+      <child link="_worktable"/>
+      <origin rpy="0 0 0" xyz="0.31057557 0.00559949 0.24"/>
+    </joint>
+    <link name="_worktable">
+      <visual>
+        <geometry>
+          <box size="0.36 0.36 0.020"/>
+        </geometry>
+        <material name="tablecolor">
+          <color rgba="0 0 0.8 1"/>
+        </material>
+      </visual>
+      <collision>
+        <geometry>
+          <box size="0.36 0.36 0.020"/>
+        </geometry>
+      </collision>
+    </link>
+    <joint name="_worktable_to_leg1" type="fixed">
+      <parent link="_worktable"/>
+      <child link="_worktable_leg1"/>
+      <origin rpy="0 0 0" xyz="0.17 0.17 -0.01"/>
+    </joint>
+    <link name="_worktable_leg1">
+      <visual>
+        <origin rpy="0 0 0" xyz="0 0 -0.115"/>
+        <geometry>
+          <box size="0.02 0.02 0.23"/>
+        </geometry>
+        <material name="leg1color">
+          <color rgba="1 1 1 1"/>
+        </material>
+      </visual>
+      <collision>
+        <origin rpy="0 0 0" xyz="0 0 -0.115"/>
+        <geometry>
+          <box size="0.02 0.02 0.23"/>
+        </geometry>
+      </collision>
+    </link>
+    <joint name="_worktable_to_leg2" type="fixed">
+      <parent link="_worktable"/>
+      <child link="_worktable_leg2"/>
+      <origin rpy="0 0 0" xyz="-0.17  0.17  -0.01"/>
+    </joint>
+    <link name="_worktable_leg2">
+      <visual>
+        <origin rpy="0 0 0" xyz="0 0 -0.115"/>
+        <geometry>
+          <box size="0.02 0.02 0.23"/>
+        </geometry>
+        <material name="leg2color">
+          <color rgba="1 1 1 1"/>
+        </material>
+      </visual>
+      <collision>
+        <origin rpy="0 0 0" xyz="0 0 -0.115"/>
+        <geometry>
+          <box size="0.02 0.02 0.23"/>
+        </geometry>
+      </collision>
+    </link>
+    <joint name="_worktable_to_leg3" type="fixed">
+      <parent link="_worktable"/>
+      <child link="_worktable_leg3"/>
+      <origin rpy="0 0 0" xyz="0.17  -0.17  -0.01"/>
+    </joint>
+    <link name="_worktable_leg3">
+      <visual>
+        <origin rpy="0 0 0" xyz="0 0 -0.115"/>
+        <geometry>
+          <box size="0.02 0.02 0.23"/>
+        </geometry>
+        <material name="leg3color">
+          <color rgba="1 1 1 1"/>
+        </material>
+      </visual>
+      <collision>
+        <origin rpy="0 0 0" xyz="0 0 -0.115"/>
+        <geometry>
+          <box size="0.02 0.02 0.23"/>
+        </geometry>
+      </collision>
+    </link>
+    <joint name="_worktable_to_leg4" type="fixed">
+      <parent link="_worktable"/>
+      <child link="_worktable_leg4"/>
+      <origin rpy="0 0 0" xyz="-0.17  -0.17  -0.01"/>
+    </joint>
+    <link name="_worktable_leg4">
+      <visual>
+        <origin rpy="0 0 0" xyz="0 0 -0.115"/>
+        <geometry>
+          <box size="0.02 0.02 0.23"/>
+        </geometry>
+        <material name="leg4color">
+          <color rgba="1 1 1 1"/>
+        </material>
+      </visual>
+      <collision>
+        <origin rpy="0 0 0" xyz="0 0 -0.115"/>
+        <geometry>
+          <box size="0.02 0.02 0.23"/>
+        </geometry>
+      </collision>
+    </link>
+-->
   </xacro:macro>
 </robot>
